File: hardware/immersion-controller-power/immersion-controller.kicad_pcb (KiCad board)
At the start: 2 copper layers, 130.5 x 73.6 mm, 31 parts, among them J1 MCU, J6 HEATER-E, J7 HEATER-N, J8 HEATER-L, J9 MAINS_IN, K3 HEATER-BOTTOM, K4 HEATER-TOP, Q4 2N3904, Q5 2N3904, U10 PC817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

Commit message: SPST Relay
Parts:
- J1: footprint Connector_PinHeader_1.27mm:PinHeader_1x04_P1.27mm_Horizontal -> Connector_PinHeader_2.54mm:PinHeader_1x04_P2.54mm_Horizontal
- K3, K4: footprint Relay_THT:Relay_SPDT_RAYEX-L90S -> Relay_THT:Relay_SPST_RAYEX-L90A
- moved J1 2.57 mm to (22.9, 131.4)
Routing:
- net Net-(K3-Pad11): track 68.7 -> 0.00 mm
- net MAINSIN_L: track 96.2 -> 156.1 mm
- net Net-(J8-Pin_2): track 71.8 -> 31.4 mm
- net Net-(J8-Pin_1): track 62.6 -> 50.4 mm
- net GND: track 228.9 -> 220.7 mm
- net +3.3V: track 19.3 -> 18.2 mm
- net RELAY_TOP: track 99.1 -> 98.2 mm
- net RELAY_BOTTOM: track 127.0 -> 127.5 mm
- net (no net): vias 6 -> 4
