File: hardware/immersion-controller-power/immersion-controller.kicad_sch (KiCad schematic)
At the start: 1 part, among them J1 MCU

Commit message: SPST Relay
Parts:
- J1: footprint Connector_PinHeader_1.27mm:PinHeader_1x04_P1.27mm_Horizontal -> Connector_PinHeader_2.54mm:PinHeader_1x04_P2.54mm_Horizontal
Changed lines of the file:
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@@
       (effects (font (size 1.27 1.27)))
     )
-    (property "Footprint" "Connector_PinHeader_1.27mm:PinHeader_1x04_P1.27mm_Horizontal" (at 156.464 52.07 0)
+    (property "Footprint" "Connector_PinHeader_2.54mm:PinHeader_1x04_P2.54mm_Horizontal" (at 156.464 52.07 0)
       (effects (font (size 1.27 1.27)) hide)
     )
