File: hardware/immersion-controller-power/output.kicad_sch (KiCad schematic)
At the start: 20 parts, among them J6 HEATER-L, J8 HEATER-E, J9 HEATER-N, J9 MAINS_IN, K1 HEATER-TOP, K2 HEATER-BOTTOM, Q1 2N3904, Q2 2N3904, U6 PC817, U7 PC817

Commit message: SPST Relay
Parts:
- K1, K2: footprint Relay_THT:Relay_SPDT_RAYEX-L90S -> Relay_THT:Relay_SPST_RAYEX-L90A; symbol Relay:RAYEX-L90S -> Relay:RAYEX-L90A
Connections:
- net MAINSIN_L: now also K1.13A, K1.13B, K2.13A, K2.13B; no longer K1.11
Changed lines of the file:
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@@
   (junction (at 115.57 82.042) (diameter 0) (color 0 0 0 0)
+  )
+  (junction (at 180.34 96.012) (diameter 0) (color 0 0 0 0)
   )
   (junction (at 115.57 43.434) (diameter 0) (color 0 0 0 0)
@@
     (stroke (width 0) (type default))
   )
-  (wire (pts (xy 174.244 41.91) (xy 163.322 41.91))
-    (stroke (width 1) (type default) (color 194 0 0 1))
-  )
   (wire (pts (xy 128.016 64.262) (xy 128.016 68.834))
     (stroke (width 0) (type default))
@@
     (stroke (width 1) (type default) (color 0 132 0 1))
   )
-  (wire (pts (xy 165.608 121.158) (xy 165.354 121.158))
+  (wire (pts (xy 180.34 121.158) (xy 165.354 121.158))
     (stroke (width 1) (type default) (color 194 0 0 1))
   )
@@
     (stroke (width 0) (type default))
   )
-  (wire (pts (xy 163.322 41.91) (xy 163.322 46.482))
-    (stroke (width 1) (type default) (color 194 0 0 1))
-  )
   (wire (pts (xy 180.34 71.374) (xy 165.862 71.374))
     (stroke (width 1) (type default) (color 194 0 0 1))
@@
     (stroke (width 1) (type default) (color 0 0 132 1))
   )
-  (wire (pts (xy 174.244 41.91) (xy 174.244 121.412))
-    (stroke (width 1) (type default) (color 194 0 0 1))
-  )
   (wire (pts (xy 186.69 38.608) (xy 168.402 38.608))
     (stroke (width 1) (type default) (color 194 0 0 1))
@@
     (stroke (width 0) (type default))
   )
-  (wire (pts (xy 165.608 121.158) (xy 165.608 121.412))
+  (wire (pts (xy 180.34 121.158) (xy 180.34 96.012))
     (stroke (width 1) (type default) (color 194 0 0 1))
   )
@@
   )
   (wire (pts (xy 180.34 71.374) (xy 180.34 96.012))
-    (stroke (width 1) (type default) (color 194 0 0 1))
-  )
-  (wire (pts (xy 174.244 121.412) (xy 165.608 121.412))
     (stroke (width 1) (type default) (color 194 0 0 1))
   )
@@
     )
   )
-  (netclass_flag "" (length 2.54) (shape round) (at 174.244 45.212 0) (fields_autoplaced)
-    (effects (font (size 1.27 1.27)) (justify left bottom))
-    (property "Netclass" "MAINS" (at 174.9425 42.672 0)
-      (effects (font (size 1.27 1.27) italic) (justify left) hide)
-    )
-    (property "Netclass" "" (at 174.9425 44.1325 0)
-      (effects (font (size 1.27 1.27) italic) (justify left))
-    )
-  )
   (symbol (lib_id "Device:LED") (at 128.016 49.784 270) (unit 1)
     (in_bom yes) (on_board yes) (dnp no) (fields_autoplaced)
@@
     )
   )
-  (symbol (lib_id "Relay:RAYEX-L90S") (at 160.782 56.642 0) (unit 1)
+  (symbol (lib_id "Relay:RAYEX-L90A") (at 160.782 56.642 0) (unit 1)
     (in_bom yes) (on_board yes) (dnp no)
     (property "Reference" "K1" (at 151.638 53.086 0)
@@
       (effects (font (size 1.27 1.27)) (justify left))
     )
-    (property "Footprint" "Relay_THT:Relay_SPDT_RAYEX-L90S" (at 172.212 57.912 0)
-      (effects (font (size 1.27 1.27)) (justify left) hide)
-    )
-    (property "Datasheet" "https://a3.sofastcdn.com/attachment/7jioKBjnRiiSrjrjknRiwS77gwbf3zmp/L90-SERIES.pdf" (at 177.292 60.452 0)
-      (effects (font (size 1.27 1.27)) (justify left) hide)
-    )
-    (pin "11")
-    (pin "12")
+    (property "Footprint" "Relay_THT:Relay_SPST_RAYEX-L90A" (at 172.212 57.912 0)
+      (effects (font (size 1.27 1.27)) (justify left) hide)
+    )
+    (property "Datasheet" "https://a3.sofastcdn.com/attachment/7jioKBjnRiiSrjrjknRiwS77gwbf3zmp/L90-SERIES.pdf" (at 178.562 60.452 0)
+      (effects (font (size 1.27 1.27)) (justify left) hide)
+    )
+    (pin "13A")
+    (pin "13B")
     (pin "14")
     (pin "A1")
@@
     )
   )
-  (symbol (lib_id "Relay:RAYEX-L90S") (at 160.274 108.712 0) (unit 1)
+  (symbol (lib_id "Relay:RAYEX-L90A") (at 160.274 108.712 0) (unit 1)
     (in_bom yes) (on_board yes) (dnp no)
     (property "Reference" "K2" (at 150.622 105.156 0)
@@
       (effects (font (size 1.27 1.27)) (justify left))
     )
-    (property "Footprint" "Relay_THT:Relay_SPDT_RAYEX-L90S" (at 171.704 109.982 0)
-      (effects (font (size 1.27 1.27)) (justify left) hide)
-    )
-    (property "Datasheet" "https://a3.sofastcdn.com/attachment/7jioKBjnRiiSrjrjknRiwS77gwbf3zmp/L90-SERIES.pdf" (at 176.784 112.522 0)
-      (effects (font (size 1.27 1.27)) (justify left) hide)
-    )
-    (pin "11")
-    (pin "12")
+    (property "Footprint" "Relay_THT:Relay_SPST_RAYEX-L90A" (at 171.704 109.982 0)
+      (effects (font (size 1.27 1.27)) (justify left) hide)
+    )
+    (property "Datasheet" "https://a3.sofastcdn.com/attachment/7jioKBjnRiiSrjrjknRiwS77gwbf3zmp/L90-SERIES.pdf" (at 178.054 112.522 0)
+      (effects (font (size 1.27 1.27)) (justify left) hide)
+    )
+    (pin "13A")
+    (pin "13B")
     (pin "14")
     (pin "A1")
