File: hardware/immersion-controller-power/output.kicad_sch (KiCad schematic)
At the start: 20 parts, among them J6 HEATER-L, J8 HEATER-E, J9 HEATER-N, J9 MAINS_IN, K1 HEATER-TOP, K2 HEATER-BOTTOM, Q1 2N3904, Q2 2N3904, U6 PC817, U7 PC817

Commit message: debugged prototype
Parts:
- D1, D2: footprint Diode_SMD:D_1210_3225Metric_Pad1.42x2.65mm_HandSolder -> LED_THT:LED_D5.0mm_Clear
- K1, K2: footprint Relay_THT:Relay_SPDT_RAYEX-L90S -> Relay_THT:Relay_SPDT_RAYEX-L90; symbol Relay:RAYEX-L90S -> Relay:RAYEX-L90
- Q1, Q2: value 2N3904 -> MMBT3904; symbol Transistor_BJT:2N3904 -> Transistor_BJT:MMBT3904
Connections:
- net GND: now also Q1.2 (E), Q2.2 (E); no longer Q1.1 (E), Q2.1 (E), R1.1, R4.1
- net MAINSIN_L: now also K1.11B; no longer K1.11
- net RELAY_BOTTOM: no longer U7.1
- net RELAY_TOP: no longer U6.1
- net VCC: now also D1.2 (A), D2.2 (A); no longer D1.1 (K), D2.1 (K)
- net at R3.1: now also D2.1 (K); no longer D2.2 (A)
- net at R6.1: now also D1.1 (K); no longer D1.2 (A)
- net at K1.12: now also K2.11B; no longer K2.11
- net at R2.2: now also Q1.1 (B); no longer Q1.2 (B)
- net at R5.2: now also Q2.1 (B); no longer Q2.2 (B)
- new net: R1.1, U6.1
- new net: R4.1, U7.1
- no-connect marks 0 -> 3
Other:
- moved on the sheet: D1, D2, R1, R4

Commit message: Initial Prototype results
Parts:
- removed J9: MAINS_IN, TerminalBlock_Dinkle:TerminalBlock_Dinkle_DT-55-B01X-03_P10.00mm, symbol Connector:Screw_Terminal_01x03
- D3, D4: value 1N4007 -> US1M; footprint Diode_SMD:D_1210_3225Metric -> Diode_SMD:D_SMA; symbol Diode:1N4007 -> Diode:US1M
Connections:
- net MAINSIN_L: now also K2.11B; no longer K1.11B
- net at K1.12: no longer K2.11B
- net at K1.14: now also J6.2 (Pin_2); no longer J6.1 (Pin_1)
- net at K2.14: now also J6.1 (Pin_1); no longer J6.2 (Pin_2)
- net at K2.12: now also K1.11B
- net VCC renamed +3.3V
