File: hardware/immersion-controller-power/psu.kicad_sch (KiCad schematic)
At the start: 10 parts, among them U8 AMS1117-3.3

Commit message: debugged prototype
Parts:
- removed D5: LED, Diode_SMD:D_1210_3225Metric_Pad1.42x2.65mm_HandSolder, symbol Device:LED
- added D1: LED, LED_THT:LED_D5.0mm_Clear, symbol Device:LED
- F2: value 1A -> 500 mA; footprint Fuse:Fuseholder_Littelfuse_100_series_5x20mm -> TE5:FUSE_BK_PCE-5-R
Connections:
- net GND: now also D1.1 (K)
- net at R7.2: now also D1.2 (A)
Changed lines of the file:
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@@
       (effects (font (size 1.27 1.27)))
     )
-    (property "Value" "1A" (at 85.09 85.09 90)
-      (effects (font (size 1.27 1.27)))
-    )
-    (property "Footprint" "Fuse:Fuseholder_Littelfuse_100_series_5x20mm" (at 85.09 88.9 90)
+    (property "Value" "500 mA" (at 85.09 85.09 90)
+      (effects (font (size 1.27 1.27)))
+    )
+    (property "Footprint" "TE5:FUSE_BK_PCE-5-R" (at 85.09 88.9 90)
       (effects (font (size 1.27 1.27)) hide)
     )
@@
   (symbol (lib_id "Device:LED") (at 163.576 102.616 90) (unit 1)
     (in_bom yes) (on_board yes) (dnp no) (fields_autoplaced)
-    (property "Reference" "D5" (at 166.624 103.5685 90)
+    (property "Reference" "D1" (at 167.64 102.9335 90)
       (effects (font (size 1.27 1.27)) (justify right))
     )
-    (property "Value" "LED" (at 166.624 106.1085 90)
+    (property "Value" "LED" (at 167.64 105.4735 90)
       (effects (font (size 1.27 1.27)) (justify right))
     )
-    (property "Footprint" "Diode_SMD:D_1210_3225Metric_Pad1.42x2.65mm_HandSolder" (at 163.576 102.616 0)
+    (property "Footprint" "LED_THT:LED_D5.0mm_Clear" (at 163.576 102.616 0)
       (effects (font (size 1.27 1.27)) hide)
     )
@@
     (instances
       (project "immersion-controller"
-        (path "/bd6e6743-d7bb-4018-a688-d589a8d21d49"
-          (reference "D5") (unit 1)
-        )
         (path "/bd6e6743-d7bb-4018-a688-d589a8d21d49/be0c28f2-d92a-481d-9fa0-7af2af8cc7a7"
           (reference "D1") (unit 1)

Commit message: Initial Prototype results
Parts:
- C1: footprint Capacitor_THT:C_Rect_L10.0mm_W3.0mm_P7.50mm_MKS4 -> Capacitor_THT:C_Rect_L11.5mm_W5.0mm_P10.00mm_MKT
- C3: footprint Capacitor_SMD:C_0805_2012Metric -> Capacitor_SMD:C_1206_3216Metric_Pad1.33x1.80mm_HandSolder
Changed lines of the file:
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@@
       (effects (font (size 1.27 1.27)) (justify left))
     )
-    (property "Footprint" "Capacitor_THT:C_Rect_L10.0mm_W3.0mm_P7.50mm_MKS4" (at 111.7092 97.282 0)
+    (property "Footprint" "Capacitor_THT:C_Rect_L11.5mm_W5.0mm_P10.00mm_MKT" (at 111.7092 97.282 0)
       (effects (font (size 1.27 1.27)) hide)
     )
@@
       (effects (font (size 1.27 1.27)) (justify left))
     )
-    (property "Footprint" "Capacitor_SMD:C_0805_2012Metric" (at 199.0852 102.108 0)
+    (property "Footprint" "Capacitor_SMD:C_1206_3216Metric_Pad1.33x1.80mm_HandSolder" (at 199.0852 102.108 0)
       (effects (font (size 1.27 1.27)) hide)
     )
