File: hardware/immersion-controller-mcu/immersion-controller.kicad_sch (KiCad schematic)
At the start: 1 part, among them J7 MCU

Commit message: Initial Prototype results
Connections:
- net +3.3V: now also J7.3 (Pin_3); no longer J7.1 (Pin_1)
- net RELAY_BOTTOM: now also J7.1 (Pin_1); no longer J7.3 (Pin_3)
Other:
- moved on the sheet: J7
Changed lines of the file:
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@@
 (kicad_sch (version 20230121) (generator eeschema)
   (paper "A4")
-  (wire (pts (xy 147.066 43.942) (xy 147.066 45.72))
+  (wire (pts (xy 144.78 35.56) (xy 147.32 35.56))
     (stroke (width 0) (type default))
   )
-  (wire (pts (xy 144.272 38.862) (xy 147.32 38.862))
+  (wire (pts (xy 144.78 43.18) (xy 147.32 43.18))
     (stroke (width 0) (type default))
   )
-  (wire (pts (xy 144.272 43.942) (xy 147.066 43.942))
+  (wire (pts (xy 144.78 38.1) (xy 147.32 38.1))
     (stroke (width 0) (type default))
   )
-  (wire (pts (xy 144.272 41.402) (xy 147.32 41.402))
+  (wire (pts (xy 144.78 40.64) (xy 170.18 40.64))
     (stroke (width 0) (type default))
   )
-  (wire (pts (xy 146.05 31.496) (xy 146.05 36.322))
+  (wire (pts (xy 170.18 38.1) (xy 170.18 40.64))
     (stroke (width 0) (type default))
   )
-  (wire (pts (xy 146.05 36.322) (xy 144.272 36.322))
+  (wire (pts (xy 147.32 43.18) (xy 147.32 45.72))
     (stroke (width 0) (type default))
   )
@@
     (effects (font (size 1.27 1.27)) (justify left top))
   )
-  (global_label "RELAY_TOP" (shape input) (at 147.32 38.862 0) (fields_autoplaced)
+  (global_label "RELAY_TOP" (shape input) (at 147.32 38.1 0) (fields_autoplaced)
     (effects (font (size 1.27 1.27)) (justify left))
-    (property "Intersheetrefs" "${INTERSHEET_REFS}" (at 160.3858 38.862 0)
+    (property "Intersheetrefs" "${INTERSHEET_REFS}" (at 160.3858 38.1 0)
       (effects (font (size 1.27 1.27)) (justify left) hide)
     )
   )
-  (global_label "RELAY_BOTTOM" (shape input) (at 147.32 41.402 0) (fields_autoplaced)
+  (global_label "RELAY_BOTTOM" (shape input) (at 147.32 35.56 0) (fields_autoplaced)
     (effects (font (size 1.27 1.27)) (justify left))
-    (property "Intersheetrefs" "${INTERSHEET_REFS}" (at 164.1353 41.402 0)
+    (property "Intersheetrefs" "${INTERSHEET_REFS}" (at 164.1353 35.56 0)
       (effects (font (size 1.27 1.27)) (justify left) hide)
     )
   )
-  (symbol (lib_id "power:+3.3V") (at 146.05 31.496 0) (unit 1)
+  (symbol (lib_id "power:+3.3V") (at 170.18 38.1 0) (unit 1)
     (in_bom yes) (on_board yes) (dnp no) (fields_autoplaced)
-    (property "Reference" "#PWR01" (at 146.05 35.306 0)
+    (property "Reference" "#PWR01" (at 170.18 41.91 0)
       (effects (font (size 1.27 1.27)) hide)
     )
-    (property "Value" "+3.3V" (at 146.05 27.432 0)
+    (property "Value" "+3.3V" (at 170.18 34.036 0)
       (effects (font (size 1.27 1.27)))
     )
-    (property "Footprint" "" (at 146.05 31.496 0)
+    (property "Footprint" "" (at 170.18 38.1 0)
       (effects (font (size 1.27 1.27)) hide)
     )
-    (property "Datasheet" "" (at 146.05 31.496 0)
+    (property "Datasheet" "" (at 170.18 38.1 0)
       (effects (font (size 1.27 1.27)) hide)
     )
@@
     )
   )
-  (symbol (lib_id "Connector:Conn_01x04_Pin") (at 139.192 38.862 0) (unit 1)
+  (symbol (lib_id "Connector:Conn_01x04_Pin") (at 139.7 38.1 0) (unit 1)
     (in_bom yes) (on_board yes) (dnp no)
-    (property "Reference" "J7" (at 139.827 32.512 0)
+    (property "Reference" "J7" (at 140.335 31.75 0)
       (effects (font (size 1.27 1.27)))
     )
-    (property "Value" "MCU" (at 135.382 31.75 0)
+    (property "Value" "MCU" (at 135.89 30.988 0)
       (effects (font (size 1.27 1.27)))
     )
-    (property "Footprint" "Connector_PinHeader_2.54mm:PinHeader_1x04_P2.54mm_Horizontal" (at 139.192 38.862 0)
+    (property "Footprint" "Connector_PinHeader_2.54mm:PinHeader_1x04_P2.54mm_Horizontal" (at 139.7 38.1 0)
       (effects (font (size 1.27 1.27)) hide)
     )
-    (property "Datasheet" "~" (at 139.192 38.862 0)
+    (property "Datasheet" "~" (at 139.7 38.1 0)
       (effects (font (size 1.27 1.27)) hide)
     )
@@
     )
   )
-  (symbol (lib_id "power:GND") (at 147.066 45.72 0) (unit 1)
-    (in_bom yes) (on_board yes) (dnp no) (fields_autoplaced)
-    (property "Reference" "#PWR02" (at 147.066 52.07 0)
+  (symbol (lib_id "power:GND") (at 147.32 45.72 0) (unit 1)
+    (in_bom yes) (on_board yes) (dnp no)
+    (property "Reference" "#PWR02" (at 147.32 52.07 0)
       (effects (font (size 1.27 1.27)) hide)
     )
-    (property "Value" "GND" (at 147.066 50.292 0)
-      (effects (font (size 1.27 1.27)))
+    (property "Value" "GND" (at 142.24 48.768 0)
+      (effects (font (size 1.27 1.27)) (justify left))
     )
-    (property "Footprint" "" (at 147.066 45.72 0)
+    (property "Footprint" "" (at 147.32 45.72 0)
       (effects (font (size 1.27 1.27)) hide)
     )
-    (property "Datasheet" "" (at 147.066 45.72 0)
+    (property "Datasheet" "" (at 147.32 45.72 0)
       (effects (font (size 1.27 1.27)) hide)
     )
