File: hardware/immersion-controller-mcu/mcu.kicad_sch (KiCad schematic)
At the start: 17 parts, among them J1 COLD, J1 TANK-BOTTOM, J1 TANK-TOP, J4 DISPLAY, J7 RTC, SW1 RotaryEncoder_Switch, U1 ESP32-S3-DevKitC, U2 TOP, U3 BOTTOM, U4 COLD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

Commit message: Initial Prototype results
Parts:
- added J6: Conn_01x02_Pin, Connector_PinHeader_2.54mm:PinHeader_1x02_P2.54mm_Vertical, symbol Connector:Conn_01x02_Pin
- J7: footprint Connector_PinHeader_2.54mm:PinHeader_1x05_P2.54mm_Vertical -> Connector_PinHeader_2.54mm:PinHeader_1x06_P2.54mm_Vertical
Connections:
- net DISPLAY_SCL: now also U1.18 (GPIO12/ADC2_CH1); no longer U1.19 (GPIO13/ADC2_CH2)
- net DISPLAY_SDA: now also U1.19 (GPIO13/ADC2_CH2); no longer U1.18 (GPIO12/ADC2_CH1)
- net GND: now also J6.1 (Pin_1)
- net ROT_CLK: now also U1.28 (GPIO47); no longer U1.27 (GPIO21)
- net WATERTEMP_DATA: now also U1.27 (GPIO21); no longer U1.13 (GPIO3/ADC1_CH2)
- net RESET: now reaches U1.3 (CHIP_PU)
- net RESET: now also J6.2 (Pin_2)
- no-connect marks 30 -> 33
Other:
- moved on the sheet: U1
